Commit message: goal mesh works

File: src/gazebo_iris/models/goal/urdf/Goal.xacro (robot description, xacro)
@@ -1,7 +1,7 @@
 <?xml version="1.0" ?>
 <robot name="Goal" xmlns:xacro="http://www.ros.org/wiki/xacro">
-<xacro:include filename="$(find gazebo_iris)/urdf/materials.xacro" />
-<xacro:include filename="$(find gazebo_iris)/urdf/Goal.trans" />
-<xacro:include filename="$(find gazebo_iris)/urdf/Goal.gazebo" />
+<xacro:include filename="$(find gazebo_iris)/models/goal/urdf/materials.xacro" />
+<xacro:include filename="$(find gazebo_iris)/models/goal/urdf/Goal.trans" />
+<xacro:include filename="$(find gazebo_iris)/models/goal/urdf/Goal.gazebo" />
 <link name="base_link">
   <inertial>
@@ -13,5 +13,5 @@
     <origin xyz="0 0 0" rpy="0 0 0"/>
     <geometry>
-      <mesh filename="package://gazebo_iris/meshes/base_link.stl" scale="0.001 0.001 0.001"/>
+      <mesh filename="package://gazebo_iris/models/goal/meshes/base_link.stl" scale="0.001 0.001 0.001"/>
     </geometry>
     <material name="silver"/>
@@ -20,5 +20,5 @@
     <origin xyz="0 0 0" rpy="0 0 0"/>
     <geometry>
-      <mesh filename="package://gazebo_iris/meshes/base_link.stl" scale="0.001 0.001 0.001"/>
+      <mesh filename="package://gazebo_iris/models/goal/meshes/base_link.stl" scale="0.001 0.001 0.001"/>
     </geometry>
   </collision>
